File: lag-gitlab.kicad_sch (KiCad schematic)
At the start: 0 parts

Commit message: Add more fields, add some info-text to sch and pcb
Other:
- note added: "Steps to complete setting up this project: Git Submodule Setup ------------------- Make sure to check out the kicad-ptx-lib as a git submodule or KiCad will cry: $ git init . $ git submodule add git@gitlab.pengutronix.de:hardware/kicad-ptx-lib.git Add libraries to project ------------------------ Afterwards add symbol and pcb libraries to project. Setup Project Variables ----------------------- .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"
Changed lines of the file:
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@@
     (company "${company}")
     (comment 1 "${release_state}")
-    (comment 2 "${prefix}-S${type_number}-R${release}-V01-C00")
+    (comment 2 "${prefix}-S${type_number}-R${release}-V${sch_variant}-C${ci}")
     (comment 3 "hardware/${prefix}-S${type_number}_${short_desciption}")
   )
+  (text "Steps to complete setting up this project:\n\n\nGit Submodule Setup\n-------------------\n\nMake sure to check out the kicad-ptx-lib as a git submodule or KiCad will cry:\n\n$ git init .\n$ git submodule add git@gitlab.pengutronix.de:hardware/kicad-ptx-lib.git\n\n\nAdd libraries to project\n------------------------\n\nAfterwards add symbol and pcb libraries to project.\n\n\nSetup Project Variables\n-----------------------\n\n... so the title blocks are nicely filled."
+    (at 29.21 135.89 0)
+    (effects (font (size 3 3)) (justify left bottom))
+  )
   (sheet_instances
