File: candlelight-S02.kicad_pcb (KiCad board)
At the start: 2 copper layers, 0 parts

Commit message: Begin project
Other:
- board text removed: "Steps to complete setting up this PCB: * Update the PCB Layerstack * Check electrical rules * Setup minimal / default track width"
Changed lines of the file:
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@@
   (property "pcb_ci" "00")
   (property "pcb_variant" "01")
-  (property "prefix" "template")
+  (property "prefix" "candlelight")
   (property "release" "01")
   (property "release_state" "draft")
   (property "sch_ci" "00")
   (property "sch_variant" "01")
-  (property "short_desciption" "template_for_LAG_projects")
-  (property "title" "Template Project")
+  (property "short_desciption" "candlelight_fd")
+  (property "title" "Candlelight FD")
   (property "type_number" "01")
   (net 0 "")
@@
     (effects (font (size 1.5 1.5) (thickness 0.3)))
   )
-  (gr_text "Steps to complete setting up this PCB:\n\n* Update the PCB Layerstack\n* Check electrical rules\n* Setup minimal / default track width" (at 88 97) (layer "Eco1.User")
-    (effects (font (size 3 3) (thickness 0.15)) (justify left))
-  )
 )
