File: tranciver.kicad_sch (KiCad schematic)
At the start: 8 parts, among them U1 TJA1051T3

Commit message: Changes during review
Other:
- company: (none) -> ${company}
- title: (none) -> Transiver
Changed lines of the file:
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@@
 (kicad_sch (version 20230121) (generator eeschema)
   (paper "A4")
+  (title_block
+    (title "Transiver")
+    (date "2023-06-16")
+    (rev "R${release}")
+    (company "${company}")
+    (comment 1 "${release_state}")
+    (comment 2 "${prefix}-S${type_number}-R${release}-V${sch_variant}-C${sch_ci}")
+    (comment 3 "hardware/${prefix}-S${type_number}_${short_desciption}")
+  )
   (junction (at 111.76 85.09) (diameter 0) (color 0 0 0 0)
   )
@@
   (symbol (lib_id "Res_1Percent_E24_0805_125mW_-40C-90C:120R_0805_125mW_1%_E24_Chip-Resistor") (at 168.91 82.55 0) (unit 1)
     (in_bom yes) (on_board yes) (dnp yes) (fields_autoplaced)
-    (property "Reference" "R5" (at 171.45 80.645 0)
+    (property "Reference" "R5" (at 171.45 80.01 0)
       (effects (font (size 1.27 1.27)) (justify left))
     )
@@
       (effects (font (size 1.524 1.524)) hide)
     )
-    (property "DisplayValue" "120R" (at 171.45 83.185 0)
+    (property "DisplayValue" "120R" (at 171.45 82.55 0)
       (effects (font (size 1.27 1.27)) (justify left))
     )
-    (property "Package" "0805" (at 168.8846 82.6008 90)
-      (effects (font (size 0.635 0.635)) hide)
-    )
-    (property "Fit" "fit: none" (at 171.45 85.09 0)
+    (property "Package" "0805" (at 171.45 84.455 0)
+      (effects (font (size 0.635 0.635)) (justify left))
+    )
+    (property "Fit" "fit: none" (at 171.45 85.725 0)
       (effects (font (size 0.635 0.635)) (justify left))
     )
@@
   (symbol (lib_id "Res_1Percent_E24_0805_125mW_-40C-90C:120R_0805_125mW_1%_E24_Chip-Resistor") (at 168.91 133.35 0) (unit 1)
     (in_bom yes) (on_board yes) (dnp yes) (fields_autoplaced)
-    (property "Reference" "R5" (at 171.45 131.445 0)
+    (property "Reference" "R5" (at 171.45 130.81 0)
       (effects (font (size 1.27 1.27)) (justify left))
     )
@@
       (effects (font (size 1.524 1.524)) hide)
     )
-    (property "DisplayValue" "120R" (at 171.45 133.985 0)
+    (property "DisplayValue" "120R" (at 171.45 133.35 0)
       (effects (font (size 1.27 1.27)) (justify left))
     )
-    (property "Package" "0805" (at 168.8846 133.4008 90)
-      (effects (font (size 0.635 0.635)) hide)
-    )
-    (property "Fit" "fit: none" (at 171.45 135.89 0)
+    (property "Package" "0805" (at 171.45 135.255 0)
       (effects (font (size 0.635 0.635)) (justify left))
     )
+    (property "Fit" "fit: none" (at 171.45 136.525 0)
+      (effects (font (size 0.635 0.635)) (justify left))
+    )
