File: MCU.kicad_sch (KiCad schematic)
At the start: 10 parts, among them P2 CONN_01X02, U1 STM32G0B1CBT, X3 TC2030-NL, Y1 830055299

Commit message: post review fix
Parts:
- added TP4, TP5: TP1.0mm, Connector_generic:TP1.0mm, symbol generic-connectors:TP1.0mm
Connections:
- net TX: now reaches U1.29 (PA9)
- net TX: now also TP5.1
- net RX: now reaches U1.32 (PA10)
- net RX: now also TP4.1
- no-connect marks 30 -> 28
Other:
- note added: "NRST has a internal pullup ~40kΩ (see: DS13560 5.3.15 NRST input characteristics)"
Changed lines of the file:
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@@
   (no_connect (at 165.1 53.34))
   (no_connect (at 165.1 50.8))
-  (no_connect (at 67.31 46.99))
   (no_connect (at 115.57 43.18))
   (no_connect (at 115.57 49.53))
-  (no_connect (at 67.31 43.18))
   (no_connect (at 157.48 25.4))
   (no_connect (at 115.57 27.94))
@@
     (stroke (width 0) (type default))
   )
+  (wire (pts (xy 59.69 43.18) (xy 67.31 43.18))
+    (stroke (width 0) (type default))
+  )
   (wire (pts (xy 57.15 49.53) (xy 67.31 49.53))
     (stroke (width 0) (type default))
@@
   )
   (wire (pts (xy 111.76 21.59) (xy 115.57 21.59))
+    (stroke (width 0) (type default))
+  )
+  (wire (pts (xy 59.69 46.99) (xy 67.31 46.99))
     (stroke (width 0) (type default))
   )
@@
     (effects (font (size 1.27 1.27)) (justify left top))
   )
+  (text "NRST has a internal pullup ~40kΩ\n(see: DS13560 5.3.15 NRST input characteristics)"
+    (at 165.1 118.11 0)
+    (effects (font (size 1.27 1.27)) (justify left bottom))
+  )
+  (label "TX" (at 59.69 43.18 0) (fields_autoplaced)
+    (effects (font (size 1.27 1.27)) (justify left bottom))
+  )
   (label "SWCLK" (at 59.69 57.15 0) (fields_autoplaced)
     (effects (font (size 1.27 1.27)) (justify left bottom))
@@
   (label "SWCLK" (at 52.07 34.29 180) (fields_autoplaced)
     (effects (font (size 1.27 1.27)) (justify right bottom))
+  )
+  (label "RX" (at 59.69 46.99 0) (fields_autoplaced)
+    (effects (font (size 1.27 1.27)) (justify left bottom))
   )
   (label "NRST" (at 156.21 107.95 0) (fields_autoplaced)
@@
     )
   )
+  (symbol (lib_id "generic-connectors:TP1.0mm") (at 59.69 43.18 180) (unit 1)
+    (in_bom yes) (on_board yes) (dnp no)
+    (property "Reference" "TP5" (at 57.15 43.18 0)
+      (effects (font (size 0.508 0.508)))
+    )
+    (property "Value" "TP1.0mm" (at 58.42 40.64 0)
+      (effects (font (size 1.524 1.524)) hide)
+    )
+    (property "Footprint" "Connector_generic:TP1.0mm" (at 69.85 53.34 0)
+      (effects (font (size 1.524 1.524)) hide)
+    )
+    (property "Datasheet" "" (at 69.85 53.34 0)
+      (effects (font (size 1.524 1.524)) hide)
+    )
+    (property "Manufacturer" "any" (at 59.69 46.99 0)
+      (effects (font (size 1.27 1.27)) hide)
+    )
+    (property "MPN" "any" (at 59.69 45.72 0)
+      (effects (font (size 1.27 1.27)) hide)
+    )
+    (property "State" "reviewed" (at 59.69 44.45 0)
+      (effects (font (size 1.27 1.27)) hide)
+    )
+    (property "Fit" "fit: " (at 59.69 48.26 0)
+      (effects (font (size 0.635 0.635)) hide)
+    )
+    (property "Package" "SMT TP" (at 59.69 43.18 0)
+      (effects (font (size 1.27 1.27)) hide)
+    )
+    (pin "1")
+    (instances
+      (project "candleLightfd-S01"
+        (path "/e63e39d7-6ac0-4ffd-8aa3-1841a4541b55/c754f27f-d753-4109-9c59-639a39396c66"
+          (reference "TP5") (unit 1)
+        )
+      )
+    )
+  )
   (symbol (lib_id "ST:STM32G0B1CBT") (at 177.8 49.53 0) (unit 4)
     (in_bom yes) (on_board yes) (dnp no) (fields_autoplaced)
@@
         )
       )
+    )
+  )
+  (symbol (lib_id "generic-connectors:TP1.0mm") (at 59.69 46.99 180) (unit 1)
+    (in_bom yes) (on_board yes) (dnp no)
+    (property "Reference" "TP4" (at 57.15 46.99 0)
+      (effects (font (size 0.508 0.508)))
+    )
+    (property "Value" "TP1.0mm" (at 58.42 44.45 0)
+      (effects (font (size 1.524 1.524)) hide)
+    )
+    (property "Footprint" "Connector_generic:TP1.0mm" (at 69.85 57.15 0)
+      (effects (font (size 1.524 1.524)) hide)
+    )
+    (property "Datasheet" "" (at 69.85 57.15 0)
+      (effects (font (size 1.524 1.524)) hide)
+    )
+    (property "Manufacturer" "any" (at 59.69 50.8 0)
+      (effects (font (size 1.27 1.27)) hide)
+    )
+    (property "MPN" "any" (at 59.69 49.53 0)
+      (effects (font (size 1.27 1.27)) hide)
+    )
+    (property "State" "reviewed" (at 59.69 48.26 0)
+      (effects (font (size 1.27 1.27)) hide)
+    )
+    (property "Fit" "fit: " (at 59.69 52.07 0)
+      (effects (font (size 0.635 0.635)) hide)
+    )
+    (property "Package" "SMT TP" (at 59.69 46.99 0)
+      (effects (font (size 1.27 1.27)) hide)
+    )
+    (pin "1")
+    (instances
+      (project "candleLightfd-S01"
+        (path "/e63e39d7-6ac0-4ffd-8aa3-1841a4541b55/c754f27f-d753-4109-9c59-639a39396c66"
+          (reference "TP4") (unit 1)
+        )
+      )
