File: MCU.kicad_sch (KiCad schematic)
At the start: 12 parts, among them P2 CONN_01X02, U1 STM32G0B1CBT, X3 TC2030-NL, Y1 830055299

Commit message: Update lib, Fix wrong value in Crystal symbol
Parts:
- Y1: value 830055299 -> 830108313809
Changed lines of the file:
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@@
       (effects (font (size 1.27 1.27)))
     )
-    (property "Value" "830055299" (at 119.38 107.95 0)
+    (property "Value" "830108313809" (at 119.38 107.95 0)
       (effects (font (size 1.27 1.27)) hide)
     )
